File: ain_pcb/ain.sch (EAGLE design)
At the start: 18 parts, among them IC2 TINY13V-10SSU, T1 BC817, X1 XPG, X2 XPG

Commit message: Added some description and changed some information
Other:
- note added: "Copyright (C) 2014-2020 Erik Kos License: Creative Commons Attribution-ShareAlike 4.0"
- note removed: "Copyright (C) 2014-2016 Jacek Szymoniak License: Creative Commons Attribution-ShareAlike 4.0"
Changed lines of the file:
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@@
 <sheet>
 <plain>
-<text x="165.1" y="25.4" size="2.794" layer="94">Copyright (C) 2014-2016 Jacek Szymoniak
+<text x="165.1" y="25.4" size="2.794" layer="94">Copyright (C) 2014-2020 Erik Kos
 License: Creative Commons Attribution-ShareAlike 4.0</text>
 </plain>
